File: KiCAD/FermentationChamberController/FermentationChamberController.kicad_pcb (KiCad board)
At the start: 2 copper layers, 17.8 x 43.2 mm, 6 parts, among them P1 Digital, P2 Analog, P3 CONN_01X01, P4 CONN_01X01, P5 CONN_01X01, P6 CONN_01X01

Commit message: Workign on the PCB Layout, first step.
Parts:
- removed P3, P4, P5, P6: CONN_01X01, Socket_Arduino_Nano:1pin_Nano
- added D1: Diode, Diodes_THT:D_DO-15_P10.16mm_Horizontal, F.Cu at (153.7, 156.2)
- added DS1: LCD16X2, Pin_Headers:Pin_Header_Straight_1x16_Pitch2.54mm, F.Cu at (100.3, 104.1)
- added J1: Screw_Terminal_1x02, Connectors_Terminal_Blocks:TerminalBlock_WAGO-804_RM5mm_2pol, F.Cu at (81.3, 97.8)
- added J2: Screw_Terminal_1x02, Connectors_Terminal_Blocks:TerminalBlock_WAGO-804_RM5mm_2pol, F.Cu at (81.3, 73.7)
- added J3: Screw_Terminal_1x02, Connectors_Terminal_Blocks:TerminalBlock_WAGO-804_RM5mm_2pol, F.Cu at (81.3, 85.1)
- added J4: CONN_01X04, Pin_Headers:Pin_Header_Angled_1x04_Pitch2.54mm, F.Cu at (255.4, 120.8)
- added J5: CONN_01X04, Pin_Headers:Pin_Header_Angled_1x04_Pitch2.54mm, F.Cu at (215.9, 152.4)
- added Q1: TIP120, TO_SOT_Packages_THT:TO-220_Horizontal, F.Cu at (210.8, 74.9)
- added Q2: TIP120, TO_SOT_Packages_THT:TO-220_Vertical, F.Cu at (144.8, 139.7)
- added R1: 4.7K, Resistors_THT:R_Axial_DIN0207_L6.3mm_D2.5mm_P10.16mm_Horizontal, F.Cu at (115.6, 101.6)
- added R2: 1.47K, Resistors_THT:R_Axial_DIN0207_L6.3mm_D2.5mm_P10.16mm_Horizontal, F.Cu at (105.4, 96.5)
- added R3: 220, Resistors_THT:R_Axial_DIN0207_L6.3mm_D2.5mm_P10.16mm_Horizontal, F.Cu at (209.6, 127.0)
- added R4: 2K, Resistors_THT:R_Axial_DIN0207_L6.3mm_D2.5mm_P10.16mm_Horizontal, F.Cu at (184.2, 91.4)
- added R5: 1K, Resistors_THT:R_Axial_DIN0207_L6.3mm_D2.5mm_P10.16mm_Horizontal, F.Cu at (154.9, 147.3)
- added R6: 10K, Resistors_THT:R_Axial_DIN0207_L6.3mm_D2.5mm_P10.16mm_Horizontal, F.Cu at (105.4, 66.0)
- added SW1: Rotary_Encoder_Switch, Pin_Headers:Pin_Header_Straight_1x05_Pitch2.54mm, F.Cu at (95.2, 76.2)
- P1, P2: footprint Socket_Arduino_Nano:Socket_Strip_Arduino_1x15 -> Pin_Headers:Pin_Header_Angled_1x15_Pitch2.54mm
- moved P2 89.0 mm to (231.1, 116.8), turned to 0 degrees
- moved P1 69.7 mm to (194.3, 114.3), turned to 0 degrees
Other:
- board size 17.8 x 43.2 mm -> 43.2 x 17.8 mm
