File: KiCAD/FermentationChamberController/FermentationChamberController.sch (KiCad schematic (older format))
At the start: 21 parts, among them J1 G Vcc, J2 1Wire 1Wire, J3 Vcc G, J4 CONN_01X04, J5 CONN_01X04, J6 CONN_01X08, J7 CONN_01X08, J8 DC Power Supply, P1 Digital, P2 Analog, Q1 TIP120, Q2 TIP120, SW1 Rotary_Encoder_Switch

Commit message: Updates to Kicad and testing
RJ 45 connectors
bad test for wifi...
Parts:
- J6, J7: footprint (none) -> Connectors:RJ45_8
- J8: footprint (none) -> Pin_Headers:Pin_Header_Straight_1x02_Pitch1.27mm
Changed lines of the file:
@@
 $EndComp
 $Comp
-L GND #PWR4
+L GND #PWR01
 U 1 1 56D7422C
 P 2750 3500
-F 0 "#PWR4" H 2750 3250 50  0001 C CNN
+F 0 "#PWR01" H 2750 3250 50  0001 C CNN
 F 1 "GND" H 2750 3350 50  0000 C CNN
 F 2 "" H 2750 3500 50  0000 C CNN
@@
 $EndComp
 $Comp
-L GND #PWR5
+L GND #PWR02
 U 1 1 56D746ED
 P 2750 4500
-F 0 "#PWR5" H 2750 4250 50  0001 C CNN
+F 0 "#PWR02" H 2750 4250 50  0001 C CNN
 F 1 "GND" H 2750 4350 50  0000 C CNN
 F 2 "" H 2750 4500 50  0000 C CNN
@@
 $EndComp
 $Comp
-L +5V #PWR11
+L +5V #PWR03
 U 1 1 56D747E8
 P 4400 4600
-F 0 "#PWR11" H 4400 4450 50  0001 C CNN
+F 0 "#PWR03" H 4400 4450 50  0001 C CNN
 F 1 "+5V" H 4400 4740 28  0000 C CNN
 F 2 "" H 4400 4600 50  0000 C CNN
@@
 $EndComp
 $Comp
-L +3.3V #PWR12
+L +3.3V #PWR04
 U 1 1 56D74854
 P 4400 4700
-F 0 "#PWR12" H 4400 4550 50  0001 C CNN
+F 0 "#PWR04" H 4400 4550 50  0001 C CNN
 F 1 "+3.3V" H 4400 4840 28  0000 C CNN
 F 2 "" H 4400 4700 50  0000 C CNN
@@
 $EndComp
 $Comp
-L Earth #PWR14
+L Earth #PWR05
 U 1 1 591B481E
 P 5300 2400
-F 0 "#PWR14" H 5300 2150 50  0001 C CNN
+F 0 "#PWR05" H 5300 2150 50  0001 C CNN
 F 1 "Earth" H 5300 2250 50  0001 C CNN
 F 2 "" H 5300 2400 50  0001 C CNN
@@
 $EndComp
 $Comp
-L Earth #PWR3
+L Earth #PWR06
 U 1 1 591B4871
 P 2750 1700
-F 0 "#PWR3" H 2750 1450 50  0001 C CNN
+F 0 "#PWR06" H 2750 1450 50  0001 C CNN
 F 1 "Earth" H 2750 1550 50  0001 C CNN
 F 2 "" H 2750 1700 50  0001 C CNN
@@
 $EndComp
 $Comp
-L +5V #PWR7
+L +5V #PWR07
 U 1 1 591B4919
 P 2850 1700
-F 0 "#PWR7" H 2850 1550 50  0001 C CNN
+F 0 "#PWR07" H 2850 1550 50  0001 C CNN
 F 1 "+5V" H 2850 1840 50  0000 C CNN
 F 2 "" H 2850 1700 50  0001 C CNN
@@
 $EndComp
 $Comp
-L Earth #PWR8
+L Earth #PWR08
 U 1 1 591B4B94
 P 2950 2250
-F 0 "#PWR8" H 2950 2000 50  0001 C CNN
+F 0 "#PWR08" H 2950 2000 50  0001 C CNN
 F 1 "Earth" H 2950 2100 50  0001 C CNN
 F 2 "" H 2950 2250 50  0001 C CNN
@@
 $EndComp
 $Comp
-L Earth #PWR9
+L Earth #PWR09
 U 1 1 591B5084
 P 3150 1700
-F 0 "#PWR9" H 3150 1450 50  0001 C CNN
+F 0 "#PWR09" H 3150 1450 50  0001 C CNN
 F 1 "Earth" H 3150 1550 50  0001 C CNN
 F 2 "" H 3150 1700 50  0001 C CNN
@@
 $EndComp
 $Comp
-L +5V #PWR10
+L +5V #PWR010
 U 1 1 591BA361
 P 4150 2000
-F 0 "#PWR10" H 4150 1850 50  0001 C CNN
+F 0 "#PWR010" H 4150 1850 50  0001 C CNN
 F 1 "+5V" H 4150 2140 50  0000 C CNN
 F 2 "" H 4150 2000 50  0001 C CNN
@@
 $EndComp
 $Comp
-L +5V #PWR19
+L +5V #PWR011
 U 1 1 591BA55B
 P 6450 1100
-F 0 "#PWR19" H 6450 950 50  0001 C CNN
+F 0 "#PWR011" H 6450 950 50  0001 C CNN
 F 1 "+5V" H 6450 1240 50  0000 C CNN
 F 2 "" H 6450 1100 50  0001 C CNN
@@
 $EndComp
 $Comp
-L GND #PWR20
+L GND #PWR012
 U 1 1 591BA655
 P 7000 1300
-F 0 "#PWR20" H 7000 1050 50  0001 C CNN
+F 0 "#PWR012" H 7000 1050 50  0001 C CNN
 F 1 "GND" H 7000 1150 50  0000 C CNN
 F 2 "" H 7000 1300 50  0001 C CNN
@@
 $EndComp
 $Comp
-L GND #PWR17
+L GND #PWR013
 U 1 1 591BA8F3
 P 5750 1200
-F 0 "#PWR17" H 5750 950 50  0001 C CNN
+F 0 "#PWR013" H 5750 950 50  0001 C CNN
 F 1 "GND" H 5750 1050 50  0000 C CNN
 F 2 "" H 5750 1200 50  0001 C CNN
@@
 $EndComp
 $Comp
-L +5V #PWR2
+L +5V #PWR014
 U 1 1 591BB0B3
 P 2150 5550
-F 0 "#PWR2" H 2150 5400 50  0001 C CNN
+F 0 "#PWR014" H 2150 5400 50  0001 C CNN
 F 1 "+5V" H 2150 5690 50  0000 C CNN
 F 2 "" H 2150 5550 50  0001 C CNN
@@
 $EndComp
 $Comp
-L GND #PWR1
+L GND #PWR015
 U 1 1 591BB21C
 P 900 6200
-F 0 "#PWR1" H 900 5950 50  0001 C CNN
+F 0 "#PWR015" H 900 5950 50  0001 C CNN
 F 1 "GND" H 900 6050 50  0000 C CNN
 F 2 "" H 900 6200 50  0001 C CNN
@@
 $EndComp
 $Comp
-L GND #PWR6
+L GND #PWR016
 U 1 1 591BB255
 P 2800 6200
-F 0 "#PWR6" H 2800 5950 50  0001 C CNN
+F 0 "#PWR016" H 2800 5950 50  0001 C CNN
 F 1 "GND" H 2800 6050 50  0000 C CNN
 F 2 "" H 2800 6200 50  0001 C CNN
@@
 $EndComp
 $Comp
-L GND #PWR25
+L GND #PWR017
 U 1 1 591BCA6D
 P 7400 6000
-F 0 "#PWR25" H 7400 5750 50  0001 C CNN
+F 0 "#PWR017" H 7400 5750 50  0001 C CNN
 F 1 "GND" H 7400 5850 50  0000 C CNN
 F 2 "" H 7400 6000 50  0001 C CNN
@@
 $EndComp
 $Comp
-L +5V #PWR29
+L +5V #PWR018
 U 1 1 591BDC18
 P 8700 4650
-F 0 "#PWR29" H 8700 4500 50  0001 C CNN
+F 0 "#PWR018" H 8700 4500 50  0001 C CNN
 F 1 "+5V" H 8700 4790 50  0000 C CNN
 F 2 "" H 8700 4650 50  0001 C CNN
@@
 $EndComp
 $Comp
-L GND #PWR28
+L GND #PWR019
 U 1 1 591BE258
 P 8700 4350
-F 0 "#PWR28" H 8700 4100 50  0001 C CNN
+F 0 "#PWR019" H 8700 4100 50  0001 C CNN
 F 1 "GND" H 8700 4200 50  0000 C CNN
 F 2 "" H 8700 4350 50  0001 C CNN
@@
 Arduino Nano
 $Comp
-L +12V #PWR27
+L +12V #PWR020
 U 1 1 591BFE81
 P 8250 5900
-F 0 "#PWR27" H 8250 5750 50  0001 C CNN
+F 0 "#PWR020" H 8250 5750 50  0001 C CNN
 F 1 "+12V" H 8250 6040 50  0000 C CNN
 F 2 "" H 8250 5900 50  0001 C CNN
@@
 $EndComp
 $Comp
-L +12V #PWR13
+L +12V #PWR021
 U 1 1 592790DF
 P 4550 4500
-F 0 "#PWR13" H 4550 4350 50  0001 C CNN
+F 0 "#PWR021" H 4550 4350 50  0001 C CNN
 F 1 "+12V" H 4550 4640 50  0000 C CNN
 F 2 "" H 4550 4500 50  0001 C CNN
@@
 F 0 "J6" H 6050 4850 50  0000 C CNN
 F 1 "CONN_01X08" V 6150 4400 50  0000 C CNN
-F 2 "" H 6050 4400 50  0001 C CNN
+F 2 "Connectors:RJ45_8" H 6050 4400 50  0001 C CNN
 F 3 "" H 6050 4400 50  0001 C CNN
 	1    6050 4400
@@
 F 0 "J7" H 6550 4850 50  0000 C CNN
 F 1 "CONN_01X08" V 6650 4400 50  0000 C CNN
-F 2 "" H 6550 4400 50  0001 C CNN
+F 2 "Connectors:RJ45_8" H 6550 4400 50  0001 C CNN
 F 3 "" H 6550 4400 50  0001 C CNN
 	1    6550 4400
@@
 $EndComp
 $Comp
-L +12V #PWR15
+L +12V #PWR022
 U 1 1 59279911
 P 5550 4050
-F 0 "#PWR15" H 5550 3900 50  0001 C CNN
+F 0 "#PWR022" H 5550 3900 50  0001 C CNN
 F 1 "+12V" H 5550 4190 50  0000 C CNN
 F 2 "" H 5550 4050 50  0001 C CNN
@@
 $EndComp
 $Comp
-L GND #PWR16
+L GND #PWR023
 U 1 1 59279A01
 P 5700 4150
-F 0 "#PWR16" H 5700 3900 50  0001 C CNN
+F 0 "#PWR023" H 5700 3900 50  0001 C CNN
 F 1 "GND" H 5700 4000 50  0000 C CNN
 F 2 "" H 5700 4150 50  0001 C CNN
@@
 $EndComp
 $Comp
-L +12V #PWR26
+L +12V #PWR024
 U 1 1 59279AF7
 P 7450 4750
-F 0 "#PWR26" H 7450 4600 50  0001 C CNN
+F 0 "#PWR024" H 7450 4600 50  0001 C CNN
 F 1 "+12V" H 7450 4890 50  0000 C CNN
 F 2 "" H 7450 4750 50  0001 C CNN
@@
 $EndComp
 $Comp
-L GND #PWR23
+L GND #PWR025
 U 1 1 59279B33
 P 7300 4650
-F 0 "#PWR23" H 7300 4400 50  0001 C CNN
+F 0 "#PWR025" H 7300 4400 50  0001 C CNN
 F 1 "GND" H 7300 4500 50  0000 C CNN
 F 2 "" H 7300 4650 50  0001 C CNN
@@
 $EndComp
 $Comp
-L +5V #PWR18
+L +5V #PWR026
 U 1 1 5927A2B7
 P 5850 4250
-F 0 "#PWR18" H 5850 4100 50  0001 C CNN
+F 0 "#PWR026" H 5850 4100 50  0001 C CNN
 F 1 "+5V" H 5850 4390 50  0000 C CNN
 F 2 "" H 5850 4250 50  0001 C CNN
@@
 $EndComp
 $Comp
-L +5V #PWR21
+L +5V #PWR027
 U 1 1 5927A5E7
 P 7100 4550
-F 0 "#PWR21" H 7100 4400 50  0001 C CNN
+F 0 "#PWR027" H 7100 4400 50  0001 C CNN
 F 1 "+5V" H 7100 4690 50  0000 C CNN
 F 2 "" H 7100 4550 50  0001 C CNN
@@
 F 0 "J8" H 7250 3800 50  0000 C CNN
 F 1 "DC Power Supply" V 7350 3650 50  0000 C CNN
-F 2 "" H 7250 3650 50  0001 C CNN
+F 2 "Pin_Headers:Pin_Header_Straight_1x02_Pitch1.27mm" H 7250 3650 50  0001 C CNN
 F 3 "" H 7250 3650 50  0001 C CNN
 	1    7250 3650
@@
 $EndComp
 $Comp
-L GND #PWR24
+L GND #PWR028
 U 1 1 5927C749
 P 7350 3850
-F 0 "#PWR24" H 7350 3600 50  0001 C CNN
+F 0 "#PWR028" H 7350 3600 50  0001 C CNN
 F 1 "GND" H 7350 3700 50  0000 C CNN
 F 2 "" H 7350 3850 50  0001 C CNN
@@
 $EndComp
 $Comp
-L +12V #PWR22
+L +12V #PWR029
 U 1 1 5927C8D9
 P 7150 3850
-F 0 "#PWR22" H 7150 3700 50  0001 C CNN
+F 0 "#PWR029" H 7150 3700 50  0001 C CNN
 F 1 "+12V" H 7150 3990 50  0000 C CNN
 F 2 "" H 7150 3850 50  0001 C CNN
